File: pcb/inverter-stage/inverter-stage.kicad_pcb (KiCad board)
At the start: 2 copper layers, 22 parts, among them J1 Screw_Terminal_01x02, J2 Conn_01x02, Q1 Q_NMOS_DGS, Q2 Q_NMOS_DGS, Q3 Q_NMOS_DGS, Q4 Q_NMOS_DGS, U1 IR2104, U2 IR2104, U3 L7805

Commit message: start tracing
Parts:
- added C5: C, Capacitor_THT:CP_Radial_D4.0mm_P2.00mm, F.Cu at (130.7, 30.3)
- added C6: C, Capacitor_THT:CP_Radial_D4.0mm_P2.00mm, F.Cu at (130.7, 35.9)
- added D3: LED, LED_THT:LED_D3.0mm, F.Cu at (143.8, 32.0)
- added H1: MountingHole, MountingHole:MountingHole_3.2mm_M3, F.Cu at (183.0, 31.0)
- added H2: MountingHole, MountingHole:MountingHole_3.2mm_M3, F.Cu at (176.0, 81.0)
- added H3: MountingHole, MountingHole:MountingHole_3.2mm_M3, F.Cu at (104.8, 81.0)
- added H4: MountingHole, MountingHole:MountingHole_3.2mm_M3, F.Cu at (105.0, 31.0)
- added R5: R, Resistor_THT:R_Axial_DIN0207_L6.3mm_D2.5mm_P7.62mm_Horizontal, F.Cu at (141.2, 38.1)
- R1, R2, R3, R4: value R -> 100R; footprint Resistor_THT:R_Axial_DIN0414_L11.9mm_D4.5mm_P15.24mm_Horizontal -> Resistor_THT:R_Axial_DIN0207_L6.3mm_D2.5mm_P7.62mm_Horizontal
- RV1, RV2: footprint Potentiometer_THT:Potentiometer_Alpha_RD901F-40-00D_Single_Vertical_CircularHoles -> Potentiometer_THT:Potentiometer_Vishay_T73XW_Horizontal
- moved J2 41.8 mm to (172.7, 34.0), turned to 180 degrees
- moved U3 37.4 mm to (135.9, 31.8), turned to 270 degrees
- moved RV1 37.2 mm to (121.0, 80.0), turned to 90 degrees
- moved J1 36.6 mm to (159.0, 34.0), turned to 180 degrees
- moved C4 17.7 mm to (153.7, 70.4), turned to 270 degrees
- moved A1 17.3 mm to (126.0, 71.1), turned to 180 degrees
- moved U2 15.9 mm to (141.0, 69.1)
- moved D2 15.8 mm to (151.0, 64.0)
- moved C3 15.5 mm to (134.0, 71.6)
- moved R4 10.9 mm to (160.0, 76.7)
- moved C2 10.7 mm to (153.7, 51.3), turned to 270 degrees
- moved Q3 10.7 mm to (181.9, 62.7)
- moved Q4 10.7 mm to (181.9, 75.4)
- moved Q1 9.71 mm to (181.9, 37.3)
- moved Q2 9.71 mm to (181.9, 50.0)
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Connections:
- RV1 pad 1: +5V -> Net-(A1-Pad27)
- RV2 pad 1: +5V -> Net-(A1-Pad27)
Routing:
- net LO_A: track 0.00 -> 11.2 mm
- net HO_A: track 0.00 -> 11.2 mm
- net A: track 0.00 -> 5.62 mm
- net Net-(C2-Pad1): track 0.00 -> 5.61 mm
Other:
- board outline added: 86 x 58 mm
- net class Power added: clearance 1, trace_width 7.62, via_dia 0.8, via_drill 0.4
- board text added: "Single Phase Inverter for 400W VFD"
- board text added: "v1.0 Mattias Zurkovic"

Commit message: pcb ready
Parts:
- Q1, Q2, Q3, Q4: value Q_NMOS_DGS -> Q_NMOS_GDS
- U3: value L7805 -> L7809
- moved A1 40.4 mm to (110.0, 34.0), turned to 0 degrees
Connections:
- A1 pad 27: Net-(A1-Pad27) -> +5V
- A1 pad 30: +5V -> +9V
- C6 pad 1: +5V -> +9V
- Q1 pad 1: VDD -> Net-(Q1-Pad1)
- Q1 pad 2: Net-(Q1-Pad2) -> VDD
- Q2 pad 1: A -> Net-(Q2-Pad1)
- Q2 pad 2: Net-(Q2-Pad2) -> A
- Q3 pad 1: VDD -> Net-(Q3-Pad1)
- Q3 pad 2: Net-(Q3-Pad2) -> VDD
- Q4 pad 1: B -> Net-(Q4-Pad1)
- Q4 pad 2: Net-(Q4-Pad2) -> B
- R1 pad 2: Net-(Q1-Pad2) -> Net-(Q1-Pad1)
- R2 pad 2: Net-(Q2-Pad2) -> Net-(Q2-Pad1)
- R3 pad 2: Net-(Q3-Pad2) -> Net-(Q3-Pad1)
- R4 pad 2: Net-(Q4-Pad2) -> Net-(Q4-Pad1)
- RV1 pad 1: Net-(A1-Pad27) -> +5V
- RV2 pad 1: Net-(A1-Pad27) -> +5V
- U3 pad 3: +5V -> +9V
Routing:
- net VDD: track 0.00 -> 170.1 mm
- net B: track 0.00 -> 145.2 mm
- net +5V: track 0.00 -> 98.9 mm
- net A: track 5.62 -> 93.3 mm
- net SHUTDOWN: track 0.00 -> 63.8 mm
- net SIG_A: track 0.00 -> 45.4 mm
- net SIG_B: track 0.00 -> 41.7 mm
- net MOD_INDEX: track 0.00 -> 25.5 mm
- net Net-(Q1-Pad1): track 0.00 -> 24.2 mm
- net SPEED: track 0.00 -> 18.8 mm
- net Net-(Q3-Pad1): track 0.00 -> 17.9 mm
- net Net-(Q2-Pad1): track 0.00 -> 17.6 mm
- net Net-(Q4-Pad1): track 0.00 -> 14.8 mm
- net Net-(C4-Pad1): track 0.00 -> 13.7 mm
- net HO_B: track 0.00 -> 13.6 mm
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- added copper zone on F.Cu, net GND
Other:
- net class OutPower added: clearance 0.2, trace_width 2, via_dia 0.8, via_drill 0.4
- net class Power: clearance 1 -> 0.5; trace_width 7.62 -> 3
- board text added: ":)"
- board text added: "A"
- board text added: "B"
- board text added: "B A"
- board text added: "MOD INDEX"
- board text added: "SPEED"
- board text added: "VDD"
- board text added: "VFD for Single Phase Induction Motor"
- board text removed: "Single Phase Inverter for 400W VFD"

Commit message: add gerber giles
Routing:
- net GND: track 0.00 -> 8.35 mm
- net VDD: track 170.1 -> 167.8 mm
Changed lines of the file:
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@@
     (thickness 1.6)
     (drawings 14)
-    (tracks 174)
+    (tracks 176)
     (zones 0)
     (modules 30)
@@
       (outputformat 1)
       (mirror false)
-      (drillshape 1)
+      (drillshape 0)
       (scaleselection 1)
-      (outputdirectory ""))
+      (outputdirectory "gerber/"))
   )
   (net 0 "")
@@
     (effects (font (size 1 1) (thickness 0.15)))
   )
+  (segment (start 134 55.078) (end 136.958 58.036) (width 0.25) (layer B.Cu) (net 1))
+  (segment (start 140.592 58.036) (end 140.97 57.658) (width 0.25) (layer B.Cu) (net 1))
+  (segment (start 136.958 58.036) (end 140.592 58.036) (width 0.25) (layer B.Cu) (net 1))
   (segment (start 135.89 31.75) (end 135.25 31.75) (width 0.25) (layer F.Cu) (net 2))
   (segment (start 133.829802 30.329802) (end 130.724999 30.329802) (width 0.25) (layer F.Cu) (net 2))
@@
   (segment (start 138.64 29) (end 135.89 31.75) (width 0.25) (layer F.Cu) (net 2))
   (segment (start 154 29) (end 138.64 29) (width 0.25) (layer F.Cu) (net 2))
-  (segment (start 135.89 31.75) (end 138.25 31.75) (width 0.25) (layer F.Cu) (net 2))
   (segment (start 140.97 66.67) (end 138.3 64) (width 0.25) (layer F.Cu) (net 2))
   (segment (start 140.97 69.088) (end 140.97 66.67) (width 0.25) (layer F.Cu) (net 2))

Commit message: first version complete - sent to fab
Parts:
- added C7: 0.1u, Capacitor_THT:CP_Radial_D4.0mm_P2.00mm, F.Cu at (130.0, 36.0)
- C1, C3: value CP -> 100u
- C2, C4: value CP -> 47u
- C5: value C -> 100u; footprint Capacitor_THT:CP_Radial_D4.0mm_P2.00mm -> Capacitor_THT:CP_Radial_D10.0mm_P5.00mm
- C6: value C -> 0.33u
- D1, D2: footprint Diode_THT:D_DO-15_P12.70mm_Horizontal -> Diode_THT:D_A-405_P10.16mm_Horizontal
- moved C5 38.1 mm to (165.0, 47.0), turned to 180 degrees
- moved C6 4.95 mm to (130.0, 31.0)
- moved R1 4.00 mm to (159.8, 56.6)
- moved R2 4.00 mm to (159.8, 61.7)
- moved D1 3.00 mm to (148.0, 45.0)
- moved D2 3.00 mm to (148.0, 64.0)
- moved C1 2.00 mm to (132.0, 52.6)
- moved C2 2.00 mm to (151.7, 51.3)
- moved C3 2.00 mm to (132.0, 71.6)
- moved C4 2.00 mm to (151.7, 70.4)
- moved U1 2.00 mm to (139.0, 50.0)
- moved U2 2.00 mm to (139.0, 69.1)
- moved RV2 1.00 mm to (110.0, 80.0)
Connections:
- C6 pad 1: +9V -> VDD
Routing:
- net VDD: track 167.8 -> 184.3 mm
- net A: track 93.3 -> 98.4 mm
- net LO_A: track 11.2 -> 14.8 mm
- net HO_B: track 13.6 -> 16.3 mm
- net HO_A: track 13.4 -> 16.0 mm
- net Net-(C2-Pad1): track 13.6 -> 11.2 mm
- net Net-(C4-Pad1): track 13.7 -> 11.2 mm
- net Net-(Q1-Pad1): track 24.2 -> 26.5 mm
- net LO_B: track 11.4 -> 13.5 mm
- net B: track 145.2 -> 147.2 mm
- net Net-(Q2-Pad1): track 17.6 -> 19.3 mm
- net +5V: track 98.9 -> 100.3 mm
- net SIG_B: track 41.7 -> 43.1 mm
- net SIG_A: track 45.4 -> 44.5 mm
- net SHUTDOWN: track 63.8 -> 63.0 mm
Other:
- board text added: "Singla Phase VFD"
- board text removed: "VFD for Single Phase Induction Motor"
