File: pcb/inverter-stage/inverter-stage.sch (KiCad schematic (older format))
At the start: 22 parts, among them J1 Screw_Terminal_01x02, J2 Conn_01x02, Q1 Q_NMOS_DGS, Q2 Q_NMOS_DGS, Q3 Q_NMOS_DGS, Q4 Q_NMOS_DGS, U1 IR2104, U2 IR2104, U3 L7805

Commit message: start tracing
Parts:
- added C5, C6: C, Capacitor_THT:CP_Radial_D4.0mm_P2.00mm, symbol pspice:C
- added D3: LED, LED_THT:LED_D3.0mm, symbol Device:LED
- added H1, H2, H3, H4: MountingHole, MountingHole:MountingHole_3.2mm_M3, symbol Mechanical:MountingHole
- added R5: R, Resistor_THT:R_Axial_DIN0207_L6.3mm_D2.5mm_P7.62mm_Horizontal, symbol Device:R
- R1, R2, R3, R4: value R -> 100R; footprint Resistor_THT:R_Axial_DIN0414_L11.9mm_D4.5mm_P15.24mm_Horizontal -> Resistor_THT:R_Axial_DIN0207_L6.3mm_D2.5mm_P7.62mm_Horizontal
- RV1, RV2: footprint Potentiometer_THT:Potentiometer_Alpha_RD901F-40-00D_Single_Vertical_CircularHoles -> Potentiometer_THT:Potentiometer_Vishay_T73XW_Horizontal
Connections:
- net +5V: now also C6.1, R5.1; no longer RV1.1, RV2.1
- net GND: now also C5.2, C6.2, D3.1 (K)
- net VDD: now also C5.1
- net at A1.27 (+5V): now also RV1.1, RV2.1
- new net: D3.2 (A), R5.2
- no-connect marks 22 -> 21
Other:
- moved on the sheet: RV1, RV2, U3

Commit message: pcb ready
Parts:
- removed Q1, Q2, Q3, Q4: Q_NMOS_DGS, Package_TO_SOT_THT:TO-220-3_Vertical, symbol Device:Q_NMOS_DGS
- added Q1, Q2, Q3, Q4: Q_NMOS_GDS, Package_TO_SOT_THT:TO-220-3_Vertical, symbol Device:Q_NMOS_GDS
- U3: value L7805 -> L7809
Connections:
- net +5V: now also A1.27 (+5V), RV1.1, RV2.1; no longer A1.30 (VIN), C6.1, U3.3 (OUT)
- net A: now also Q1.3 (S), Q2.2 (D)
- net B: now also Q3.3 (S), Q4.2 (D)
- net GND: now also Q2.3 (S), Q4.3 (S)
- net VDD: now also Q1.2 (D), Q3.2 (D)
- net at R1.2: now also Q1.1 (G)
- net at R2.2: now also Q2.1 (G)
- net at R3.2: now also Q3.1 (G)
- net at R4.2: now also Q4.1 (G)
- new net +9V: A1.30 (VIN), C6.1, U3.3 (OUT)
Other:
- note added: "Misc and Status"
- note added: "VFD Inverter Stage for Single Phase Induction Motors"
- moved on the sheet: A1, C1, C2, C3, C4, C5, C6, D1, D2, D3, H1, H2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

Commit message: first version complete - sent to fab
Parts:
- removed C5, C6: C, Capacitor_THT:CP_Radial_D4.0mm_P2.00mm, symbol pspice:C
- added C5: 100u, Capacitor_THT:CP_Radial_D10.0mm_P5.00mm, symbol Device:C
- added C6: 0.33u, Capacitor_THT:CP_Radial_D4.0mm_P2.00mm, symbol Device:C
- added C7: 0.1u, Capacitor_THT:CP_Radial_D4.0mm_P2.00mm, symbol Device:C
- C1, C3: value CP -> 100u
- C2, C4: value CP -> 47u
- D1, D2: footprint Diode_THT:D_DO-15_P12.70mm_Horizontal -> Diode_THT:D_A-405_P10.16mm_Horizontal
Connections:
- net +9V: now also C7.1
- net GND: now also C5.2, C6.2, C7.2
- net VDD: now also C5.1, C6.1
Other:
- moved on the sheet: J1, U3
Changed lines of the file:
@@
 F 0 "D1" H 7750 4083 50  0000 C CNN
 F 1 "D" H 7750 4174 50  0000 C CNN
-F 2 "Diode_THT:D_DO-15_P12.70mm_Horizontal" H 7750 4300 50  0001 C CNN
+F 2 "Diode_THT:D_A-405_P10.16mm_Horizontal" H 7750 4300 50  0001 C CNN
 F 3 "~" H 7750 4300 50  0001 C CNN
 	1    7750 4300
@@
 P 6400 4750
 F 0 "C1" H 6518 4796 50  0000 L CNN
-F 1 "CP" H 6518 4705 50  0000 L CNN
+F 1 "100u" H 6518 4705 50  0000 L CNN
 F 2 "Capacitor_THT:CP_Radial_D6.3mm_P2.50mm" H 6438 4600 50  0001 C CNN
 F 3 "~" H 6400 4750 50  0001 C CNN
@@
 P 8100 4750
 F 0 "C2" H 8218 4796 50  0000 L CNN
-F 1 "CP" H 8218 4705 50  0000 L CNN
+F 1 "47u" H 8218 4705 50  0000 L CNN
 F 2 "Capacitor_THT:CP_Radial_D5.0mm_P2.50mm" H 8138 4600 50  0001 C CNN
 F 3 "~" H 8100 4750 50  0001 C CNN
@@
 F 0 "D2" H 10100 4083 50  0000 C CNN
 F 1 "D" H 10100 4174 50  0000 C CNN
-F 2 "Diode_THT:D_DO-15_P12.70mm_Horizontal" H 10100 4300 50  0001 C CNN
+F 2 "Diode_THT:D_A-405_P10.16mm_Horizontal" H 10100 4300 50  0001 C CNN
 F 3 "~" H 10100 4300 50  0001 C CNN
 	1    10100 4300
@@
 P 8750 4750
 F 0 "C3" H 8868 4796 50  0000 L CNN
-F 1 "CP" H 8868 4705 50  0000 L CNN
+F 1 "100u" H 8868 4705 50  0000 L CNN
 F 2 "Capacitor_THT:CP_Radial_D6.3mm_P2.50mm" H 8788 4600 50  0001 C CNN
 F 3 "~" H 8750 4750 50  0001 C CNN
@@
 P 10450 4750
 F 0 "C4" H 10568 4796 50  0000 L CNN
-F 1 "CP" H 10568 4705 50  0000 L CNN
+F 1 "47u" H 10568 4705 50  0000 L CNN
 F 2 "Capacitor_THT:CP_Radial_D5.0mm_P2.50mm" H 10488 4600 50  0001 C CNN
 F 3 "~" H 10450 4750 50  0001 C CNN
@@
 L power:GND #PWR010
 U 1 1 61B6CC90
-P 5000 1500
-F 0 "#PWR010" H 5000 1250 50  0001 C CNN
-F 1 "GND" V 5005 1372 50  0000 R CNN
-F 2 "" H 5000 1500 50  0001 C CNN
-F 3 "" H 5000 1500 50  0001 C CNN
-	1    5000 1500
-	0    1    1    0
-$EndComp
-$Comp
-L power:VDD #PWR09
-U 1 1 61B6D2DC
-P 5000 1400
-F 0 "#PWR09" H 5000 1250 50  0001 C CNN
-F 1 "VDD" V 5015 1527 50  0000 L CNN
-F 2 "" H 5000 1400 50  0001 C CNN
-F 3 "" H 5000 1400 50  0001 C CNN
-	1    5000 1400
-	0    -1   -1   0
+P 4950 1750
+F 0 "#PWR010" H 4950 1500 50  0001 C CNN
+F 1 "GND" V 4955 1622 50  0000 R CNN
+F 2 "" H 4950 1750 50  0001 C CNN
+F 3 "" H 4950 1750 50  0001 C CNN
+	1    4950 1750
+	1    0    0    -1
 $EndComp
 $Comp
 L Regulator_Linear:L7805 U3
 U 1 1 61B72F08
-P 5350 2000
-F 0 "U3" H 5350 2242 50  0000 C CNN
-F 1 "L7809" H 5350 2151 50  0000 C CNN
-F 2 "Package_TO_SOT_THT:TO-220-3_Vertical" H 5375 1850 50  0001 L CIN
-F 3 "http://www.st.com/content/ccc/resource/technical/document/datasheet/41/4f/b3/b0/12/d4/47/88/CD00000444.pdf/files/CD00000444.pdf/jcr:content/translations/en.CD00000444.pdf" H 5350 1950 50  0001 C CNN
-	1    5350 2000
-	1    0    0    -1
-$EndComp
-Text Notes 6000 2850 0    50   ~ 0
+P 5400 2300
+F 0 "U3" H 5400 2542 50  0000 C CNN
+F 1 "L7809" H 5400 2451 50  0000 C CNN
+F 2 "Package_TO_SOT_THT:TO-220-3_Vertical" H 5425 2150 50  0001 L CIN
+F 3 "http://www.st.com/content/ccc/resource/technical/document/datasheet/41/4f/b3/b0/12/d4/47/88/CD00000444.pdf/files/CD00000444.pdf/jcr:content/translations/en.CD00000444.pdf" H 5400 2250 50  0001 C CNN
+	1    5400 2300
+	1    0    0    -1
+$EndComp
+Text Notes 6100 2950 0    50   ~ 0
 Input Power
 $Comp
@@
 L power:PWR_FLAG #FLG0101
 U 1 1 61A678AE
-P 5000 1400
-F 0 "#FLG0101" H 5000 1475 50  0001 C CNN
-F 1 "PWR_FLAG" H 5000 1573 50  0000 C CNN
-F 2 "" H 5000 1400 50  0001 C CNN
-F 3 "~" H 5000 1400 50  0001 C CNN
-	1    5000 1400
-	1    0    0    -1
-$EndComp
-Connection ~ 5000 1400
+P 5300 1450
+F 0 "#FLG0101" H 5300 1525 50  0001 C CNN
+F 1 "PWR_FLAG" H 5300 1623 50  0000 C CNN
+F 2 "" H 5300 1450 50  0001 C CNN
+F 3 "~" H 5300 1450 50  0001 C CNN
+	1    5300 1450
+	1    0    0    -1
+$EndComp
 $Comp
 L power:PWR_FLAG #FLG0102
 U 1 1 61A68D39
-P 5000 1500
-F 0 "#FLG0102" H 5000 1575 50  0001 C CNN
-F 1 "PWR_FLAG" H 5000 1673 50  0000 C CNN
-F 2 "" H 5000 1500 50  0001 C CNN
-F 3 "~" H 5000 1500 50  0001 C CNN
-	1    5000 1500
+P 5300 1750
+F 0 "#FLG0102" H 5300 1825 50  0001 C CNN
+F 1 "PWR_FLAG" H 5300 1923 50  0000 C CNN
+F 2 "" H 5300 1750 50  0001 C CNN
+F 3 "~" H 5300 1750 50  0001 C CNN
+	1    5300 1750
 	-1   0    0    1
 $EndComp
-Connection ~ 5000 1500
 Text GLabel 9350 4900 0    50   Input ~ 0
 SHUTDOWN
@@
 	1    0    0    -1
 $EndComp
-Wire Notes Line
-	4300 1150 4300 2750
-Wire Notes Line
-	4300 2750 6450 2750
-Wire Notes Line
-	6450 2750 6450 1150
-Wire Notes Line
-	4300 1150 6450 1150
 $Comp
 L Connector:Screw_Terminal_01x02 J1
 U 1 1 61B690AC
-P 5200 1400
-F 0 "J1" H 5280 1392 50  0000 L CNN
-F 1 "Screw_Terminal_01x02" H 5280 1301 50  0000 L CNN
-F 2 "TerminalBlock:TerminalBlock_Altech_AK300-2_P5.00mm" H 5200 1400 50  0001 C CNN
-F 3 "~" H 5200 1400 50  0001 C CNN
-	1    5200 1400
+P 5500 1550
+F 0 "J1" H 5580 1542 50  0000 L CNN
+F 1 "Screw_Terminal_01x02" H 5580 1451 50  0000 L CNN
+F 2 "TerminalBlock:TerminalBlock_Altech_AK300-2_P5.00mm" H 5500 1550 50  0001 C CNN
+F 3 "~" H 5500 1550 50  0001 C CNN
+	1    5500 1550
 	1    0    0    -1
 $EndComp
@@
 L power:VDD #PWR011
 U 1 1 61B740BF
-P 4750 2000
-F 0 "#PWR011" H 4750 1850 50  0001 C CNN
-F 1 "VDD" V 4765 2127 50  0000 L CNN
-F 2 "" H 4750 2000 50  0001 C CNN
-F 3 "" H 4750 2000 50  0001 C CNN
-	1    4750 2000
+P 4800 2300
+F 0 "#PWR011" H 4800 2150 50  0001 C CNN
+F 1 "VDD" V 4815 2427 50  0000 L CNN
+F 2 "" H 4800 2300 50  0001 C CNN
+F 3 "" H 4800 2300 50  0001 C CNN
+	1    4800 2300
 	0    -1   -1   0
 $EndComp
@@
 L power:GND #PWR012
 U 1 1 61B74DBF
-P 5350 2500
-F 0 "#PWR012" H 5350 2250 50  0001 C CNN
-F 1 "GND" H 5355 2327 50  0000 C CNN
-F 2 "" H 5350 2500 50  0001 C CNN
-F 3 "" H 5350 2500 50  0001 C CNN
-	1    5350 2500
-	1    0    0    -1
-$EndComp
-Wire Wire Line
-	5350 2500 5350 2300
-Connection ~ 5350 2500
-Wire Wire Line
-	5850 2500 5350 2500
-Wire Wire Line
-	4850 2500 5350 2500
-Wire Wire Line
-	5850 2000 5650 2000
-Wire Wire Line
-	5950 2000 5850 2000
-Connection ~ 5850 2000
-$Comp
-L pspice:C C6
-U 1 1 61ACF074
-P 5850 2250
-F 0 "C6" H 6028 2296 50  0000 L CNN
-F 1 "C" H 6028 2205 50  0000 L CNN
-F 2 "Capacitor_THT:CP_Radial_D4.0mm_P2.00mm" H 5850 2250 50  0001 C CNN
-F 3 "~" H 5850 2250 50  0001 C CNN
-	1    5850 2250
-	1    0    0    -1
-$EndComp
-Wire Wire Line
-	5050 2000 4850 2000
-Wire Wire Line
-	4750 2000 4850 2000
-Connection ~ 4850 2000
-$Comp
-L pspice:C C5
-U 1 1 61ACD79E
-P 4850 2250
-F 0 "C5" H 5028 2296 50  0000 L CNN
-F 1 "C" H 5028 2205 50  0000 L CNN
-F 2 "Capacitor_THT:CP_Radial_D4.0mm_P2.00mm" H 4850 2250 50  0001 C CNN
-F 3 "~" H 4850 2250 50  0001 C CNN
-	1    4850 2250
+P 5400 2600
+F 0 "#PWR012" H 5400 2350 50  0001 C CNN
+F 1 "GND" H 5405 2427 50  0000 C CNN
+F 2 "" H 5400 2600 50  0001 C CNN
+F 3 "" H 5400 2600 50  0001 C CNN
+	1    5400 2600
 	1    0    0    -1
 $EndComp
@@
 L power:+9V #PWR0101
 U 1 1 61A9CB63
-P 5950 2000
-F 0 "#PWR0101" H 5950 1850 50  0001 C CNN
-F 1 "+9V" V 5965 2128 50  0000 L CNN
-F 2 "" H 5950 2000 50  0001 C CNN
-F 3 "" H 5950 2000 50  0001 C CNN
-	1    5950 2000
+P 6000 2300
+F 0 "#PWR0101" H 6000 2150 50  0001 C CNN
+F 1 "+9V" V 6015 2428 50  0000 L CNN
+F 2 "" H 6000 2300 50  0001 C CNN
+F 3 "" H 6000 2300 50  0001 C CNN
+	1    6000 2300
 	0    1    1    0
 $EndComp
@@
 	1    0    0    -1
 $EndComp
+$Comp
+L power:VDD #PWR09
+U 1 1 61B6D2DC
+P 4950 1450
+F 0 "#PWR09" H 4950 1300 50  0001 C CNN
+F 1 "VDD" V 4965 1577 50  0000 L CNN
+F 2 "" H 4950 1450 50  0001 C CNN
+F 3 "" H 4950 1450 50  0001 C CNN
+	1    4950 1450
+	1    0    0    -1
+$EndComp
+$Comp
+L Device:C C5
+U 1 1 61A87E69
+P 4950 1600
+F 0 "C5" H 5065 1646 50  0000 L CNN
+F 1 "100u" H 5065 1555 50  0000 L CNN
+F 2 "Capacitor_THT:CP_Radial_D10.0mm_P5.00mm" H 4988 1450 50  0001 C CNN
+F 3 "~" H 4950 1600 50  0001 C CNN
+	1    4950 1600
+	1    0    0    -1
+$EndComp
+Wire Wire Line
+	4800 2300 4950 2300
+Wire Wire Line
+	5700 2300 5850 2300
+$Comp
+L Device:C C6
+U 1 1 61A902B3
+P 4950 2450
+F 0 "C6" H 5065 2496 50  0000 L CNN
+F 1 "0.33u" H 5065 2405 50  0000 L CNN
+F 2 "Capacitor_THT:CP_Radial_D4.0mm_P2.00mm" H 4988 2300 50  0001 C CNN
+F 3 "~" H 4950 2450 50  0001 C CNN
+	1    4950 2450
+	1    0    0    -1
+$EndComp
+Connection ~ 4950 2300
+Wire Wire Line
+	4950 2300 5100 2300
+$Comp
+L Device:C C7
+U 1 1 61A90E0C
+P 5850 2450
+F 0 "C7" H 5965 2496 50  0000 L CNN
+F 1 "0.1u" H 5965 2405 50  0000 L CNN
+F 2 "Capacitor_THT:CP_Radial_D4.0mm_P2.00mm" H 5888 2300 50  0001 C CNN
+F 3 "~" H 5850 2450 50  0001 C CNN
+	1    5850 2450
+	1    0    0    -1
+$EndComp
+Connection ~ 5850 2300
+Wire Wire Line
+	5850 2300 6000 2300
+Wire Wire Line
+	4950 2600 5400 2600
+Connection ~ 5400 2600
+Wire Wire Line
+	5850 2600 5400 2600
+Wire Wire Line
+	5300 1650 5300 1750
+Wire Wire Line
+	5300 1750 4950 1750
+Wire Wire Line
+	4950 1450 5300 1450
+Wire Wire Line
+	5300 1450 5300 1550
+Connection ~ 4950 1750
+Connection ~ 4950 1450
+Connection ~ 5300 1750
+Connection ~ 5300 1450
+Wire Notes Line
+	4450 1150 6550 1150
+Wire Notes Line
+	6550 1150 6550 2850
+Wire Notes Line
+	6550 2850 4450 2850
+Wire Notes Line
+	4450 2850 4450 1150
 $EndSCHEMATC
